Commit message: Add kinect-v2 model

File: eddiebot/eddiebot_description/robots/eddie_kinect_v1.urdf.xacro (robot description, xacro)
@@ -1,4 +1,4 @@
 <?xml version="1.0"?>
-<robot name="arlobot" xmlns:xacro="http://ros.org/wiki/xacro">
+<robot name="eddiebot" xmlns:xacro="http://ros.org/wiki/xacro">
   <!-- From $(find turtlebot_description)/urdf/common_properties.urdf.xacro -->
   <!-- It is required by asus_xtion_pro.urdf.xacro (primesense carmine)-->
@@ -9,5 +9,5 @@
   <xacro:include filename="$(find eddiebot_description)/urdf/stacks/camera_stand.urdf.xacro"/>
   <!-- Kinect Sensor -->
-  <xacro:include filename="$(find eddiebot_description)/urdf/sensors/kinect.urdf.xacro"/>
+  <xacro:include filename="$(find eddiebot_description)/urdf/sensors/kinect_v1.urdf.xacro"/>
   <create_base/>
   <circle_stack parent="base_link"/>

File: eddiebot/eddiebot_description/robots/eddie_primesense.urdf.xacro (robot description, xacro)
@@ -1,4 +1,4 @@
 <?xml version="1.0"?>
-<robot name="arlobot" xmlns:xacro="http://ros.org/wiki/xacro">
+<robot name="eddiebot" xmlns:xacro="http://ros.org/wiki/xacro">
   <!-- A common file to tie together all of the bits and bobs of the entire robot
   Modeled after turtlebot_description

File: eddiebot/eddiebot_description/urdf/camera_properties.urdf.xacro (robot description, xacro)
@@ -1,4 +1,4 @@
 <?xml version="1.0"?>
-<robot xmlns:xacro="http://ros.org/wiki/xacro">
+<robot xmlns:xacro="http://www.ros.org/wiki/xacro">
   <!--
     These properties must be observed by any machine
@@ -34,4 +34,4 @@
 	<!-- Test this by setting the robot's axles exactly 1 meter from a wall, start up RVIZ with the robot at 0,0,0 on the grid, -->
 	<!-- and see if the wall lines up straight with the grid line. -->
-	<xacro:property name="cam_oy" value="-0.005" />
+	<xacro:property name="cam_oy" value="0" />
 </robot>
