Commit message: Update kinect-v2 position on robot

File: eddiebot/eddiebot_description/robots/eddie_kinect_v2.urdf.xacro (robot description, xacro)
@@ -13,4 +13,4 @@
   <circle_stack parent="base_link"/>
   <camera_stand parent="plate_0_link"/>
-  <sensor_kinect_v2 parent="camera_mount_link" />
+  <sensor_kinect_v2 parent="base_link" />
 </robot>

File: eddiebot/eddiebot_description/urdf/sensors/kinect_v2.urdf.xacro (robot description, xacro)
@@ -6,5 +6,5 @@
   <xacro:property name="kinect_v2_cam_px" value="0.0975"/>
   <xacro:property name="kinect_v2_cam_py" value="0.01" />
-  <xacro:property name="kinect_v2_cam_pz" value="0" />
+  <xacro:property name="kinect_v2_cam_pz" value="0.15" />
   <!-- This is the tilt across the horizontal when looking straight at the camera. Probably important, but hard to see if it is. -->
   <xacro:property name="cam_or" value="0" />
