Commit message: Add eddiebot gazebo simulation world

File: eddiebot/eddiebot_description/urdf/stacks/create_base.urdf.xacro (robot description, xacro)
@@ -1,4 +1,5 @@
 <?xml version="1.0"?>
 <robot name="eddiebot_create_base" xmlns:xacro="http://ros.org/wiki/xacro">
+  <xacro:property name="M_PI" value="3.1415926535897931" />
   <!-- Macro for creating eddiebot base. -->
   <!-- <xacro:property name="base_x" value="0.33" /> -->
@@ -87,4 +88,8 @@
       </inertial>
       <visual>
+        <!-- <geometry>
+          <cylinder length="0.061" radius="0.05"/>
+        </geometry>
+        <origin rpy="${M_PI/2} 0 0" xyz="0 0 -0.05"/> -->
         <origin xyz="0 0 0" rpy="-1.5707 0 1.5707" />
         <geometry>
@@ -95,4 +100,10 @@
         </material>
       </visual>
+      <collision>
+        <geometry>
+          <cylinder length="0.061" radius="0.05"/>
+        </geometry>
+        <origin rpy="${M_PI/2} 0 0" xyz="0 0 -0.05"/>
+      </collision>
     </link>
     <joint name="front_caster_joint" type="fixed">
@@ -118,4 +129,10 @@
         </material>
       </visual>
+      <collision>
+        <geometry>
+          <cylinder length="0.061" radius="0.05"/>
+        </geometry>
+        <origin rpy="${M_PI/2} 0 0" xyz="0 0 -0.05"/>
+      </collision>
     </link>
     <joint name="rear_caster_joint" type="fixed">
